Commit message: Etapa 5.3-Ultimo Arreglo URDF, rviz configurado

File: robot_ws/install/scanbot_description/share/scanbot_description/urdf/scanbot_description.urdf (robot description, URDF)
Before this commit: robot ScanBot__f, 5 links, 4 joints
Links:
- link Left_Gear_link: geometry collision mesh filename=package://scanbot_description/meshes/Left_Gear_link.STL; visual mesh filename=package://scanbot_description/meshes/Left_Gear_link.STL
- link Left_Scatter_Gear_link: geometry collision mesh filename=package://scanbot_description/meshes/Left_Scatter_Gear_link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; visual mesh filename=package://scanbot_description/meshes/Left_Scatter_Gear_link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
- link Rigth_Gear_link: geometry collision mesh filename=package://scanbot_description/meshes/Rigth_Gear_link.STL; visual mesh filename=package://scanbot_description/meshes/Rigth_Gear_link.STL
- link Rigth_Scatter_Gear_link: geometry collision mesh filename=package://scanbot_description/meshes/Rigth_Scatter_Gear_lin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; visual mesh filename=package://scanbot_description/meshes/Rigth_Scatter_Gear_lin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
- link base_link: geometry collision mesh filename=package://scanbot_description/meshes/base_link.STL; visual mesh filename=package://scanbot_description/meshes/base_link.STL
