Commit message: Etapa 5.3-Ultimo Arreglo URDF, rviz configurado

File: robot_ws/install/scanbot_description/share/scanbot_description/urdf/scanbot_description.urdf.xacro (robot description, xacro)
@@ -103,5 +103,5 @@
   <!-- RIGHT GEAR LINK                                        -->
   <!-- ====================================================== -->
-  <link name="Rigth_Gear_link">
+  <link name="Right_Gear_link">
     <inertial>
       <origin
@@ -121,22 +121,22 @@
       <geometry>
         <mesh
-          filename="package://scanbot_description/meshes/Rigth_Gear_link.STL"
-          scale="1 1 1"/>
-      </geometry>
-      <material name="pink">
-        <color rgba="1 0.71765 0.96863 1"/>
-      </material>
-    </visual>
-    <collision>
-      <origin xyz="0 0 0" rpy="0 0 0"/>
-      <geometry>
-        <mesh
-          filename="package://scanbot_description/meshes/Rigth_Gear_link.STL"
-          scale="1 1 1"/>
-      </geometry>
-    </collision>
-  </link>
-  <joint
-    name="Rigth_Gear_joint"
+          filename="package://scanbot_description/meshes/Right_Gear_link.STL"
+          scale="1 1 1"/>
+      </geometry>
+      <material name="pink">
+        <color rgba="1 0.71765 0.96863 1"/>
+      </material>
+    </visual>
+    <collision>
+      <origin xyz="0 0 0" rpy="0 0 0"/>
+      <geometry>
+        <mesh
+          filename="package://scanbot_description/meshes/Right_Gear_link.STL"
+          scale="1 1 1"/>
+      </geometry>
+    </collision>
+  </link>
+  <joint
+    name="Right_Gear_joint"
     type="continuous">
     <origin
@@ -144,5 +144,5 @@
       rpy="1.5708 0 0"/>
     <parent link="base_link"/>
-    <child link="Rigth_Gear_link"/>
+    <child link="Right_Gear_link"/>
     <axis xyz="0 0 1"/>
     <limit
@@ -209,5 +209,5 @@
   <!-- RIGHT SCATTER GEAR                                     -->
   <!-- ====================================================== -->
-  <link name="Rigth_Scatter_Gear_link">
+  <link name="Right_Scatter_Gear_link">
     <inertial>
       <origin
@@ -227,22 +227,22 @@
       <geometry>
         <mesh
-          filename="package://scanbot_description/meshes/Rigth_Scatter_Gear_link.STL"
-          scale="1 1 1"/>
-      </geometry>
-      <material name="pink">
-        <color rgba="1 0.71765 0.96863 1"/>
-      </material>
-    </visual>
-    <collision>
-      <origin xyz="0 0 0" rpy="0 0 0"/>
-      <geometry>
-        <mesh
-          filename="package://scanbot_description/meshes/Rigth_Scatter_Gear_link.STL"
-          scale="1 1 1"/>
-      </geometry>
-    </collision>
-  </link>
-  <joint
-    name="Rigth_Scatter_Gear_joint"
+          filename="package://scanbot_description/meshes/Right_Scatter_Gear_link.STL"
+          scale="1 1 1"/>
+      </geometry>
+      <material name="pink">
+        <color rgba="1 0.71765 0.96863 1"/>
+      </material>
+    </visual>
+    <collision>
+      <origin xyz="0 0 0" rpy="0 0 0"/>
+      <geometry>
+        <mesh
+          filename="package://scanbot_description/meshes/Right_Scatter_Gear_link.STL"
+          scale="1 1 1"/>
+      </geometry>
+    </collision>
+  </link>
+  <joint
+    name="Right_Scatter_Gear_joint"
     type="continuous">
     <origin
@@ -250,5 +250,5 @@
       rpy="1.5708 -0.082932 0"/>
     <parent link="base_link"/>
-    <child link="Rigth_Scatter_Gear_link"/>
+    <child link="Right_Scatter_Gear_link"/>
     <axis xyz="0 0 1"/>
     <limit

Commit message: Etapa 6. Empezar a pasar /topicos esp32 a rviz

File: robot_ws/install/scanbot_description/share/scanbot_description/urdf/scanbot_description.urdf.xacro (robot description, xacro)
@@ -8,5 +8,6 @@
     <parent link="base_footprint"/>
     <child link="base_link"/>
-    <origin xyz="0 0 0" rpy="0 0 0"/>
+    <!-- Altura del robot respecto al suelo -->
+    <origin xyz="0 0 0.03" rpy="0 0 0"/>
   </joint>
   <!-- ====================================================== -->
@@ -259,3 +260,73 @@
       friction="0.1"/>
   </joint>
+  <!-- ====================================================== -->
+  <!-- LIDAR LINK                                              -->
+  <!-- ====================================================== -->
+  <link name="laser_link">
+    <visual>
+      <origin xyz="0 0 0" rpy="0 0 0"/>
+      <geometry>
+        <cylinder radius="0.003" length="0.004"/>
+      </geometry>
+      <material name="blue">
+        <color rgba="0 0 1 1"/>
+      </material>
+    </visual>
+  </link>
+  <joint name="laser_joint" type="fixed">
+    <parent link="base_link"/>
+    <child link="laser_link"/>
+    <!-- AJUSTAR POSICIÓN -->
+    <origin xyz="0.10 0 0.10" rpy="0 0 0"/>
+  </joint>
+  <!-- ====================================================== -->
+  <!-- IMU LINK                                                -->
+  <!-- ====================================================== -->
+  <link name="imu_link">
+    <visual>
+      <origin xyz="0 0 0" rpy="0 0 0"/>
+      <geometry>
+        <box size="0.002 0.002 0.001"/>
+      </geometry>
+      <material name="green">
+        <color rgba="0 1 0 1"/>
+      </material>
+    </visual>
+  </link>
+  <joint name="imu_joint" type="fixed">
+    <parent link="base_link"/>
+    <child link="imu_link"/>
+    <!-- AJUSTAR POSICIÓN -->
+    <origin xyz="0 0 0.03" rpy="0 0 0"/>
+  </joint>
+  <!-- ====================================================== -->
+  <!-- CAMERA LINK                                             -->
+  <!-- ====================================================== -->
+  <link name="camera_link">
+    <visual>
+      <origin xyz="0 0 0" rpy="0 0 0"/>
+      <geometry>
+        <box size="0.004 0.004 0.004"/>
+      </geometry>
+      <material name="red">
+        <color rgba="1 0 0 1"/>
+      </material>
+    </visual>
+  </link>
+  <joint name="camera_joint" type="fixed">
+    <parent link="base_link"/>
+    <child link="camera_link"/>
+    <!-- AJUSTAR POSICIÓN -->
+    <origin xyz="0.08 0 0.12" rpy="0 0 0"/>
+  </joint>
+  <!-- ====================================================== -->
+  <!-- CAMERA OPTICAL LINK                                     -->
+  <!-- ====================================================== -->
+  <link name="camera_optical_link"/>
+  <joint name="camera_optical_joint" type="fixed">
+    <parent link="camera_link"/>
+    <child link="camera_optical_link"/>
+    <!-- ROS Optical Frame Convention -->
+    <origin xyz="0 0 0" rpy="-1.5708 0 -1.5708"/>
+  </joint>
 </robot>
